File: LinkSocket.kicad_sch (KiCad schematic)
At the start: 4 parts, among them J201 2x05_Horizontal

Commit message: Update
Parts:
- C10: renamed from C201; Id (none) -> Capacitor:${SYMBOL_NAME}
- J5: renamed from J201; Id (none) -> Header:${SYMBOL_NAME}; Rating (none) -> 1A
- R5: renamed from R201; Id (none) -> Resistor:${SYMBOL_NAME}
- U3: renamed from U201; Id (none) -> RS485:${SYMBOL_NAME}
Other:
- company: Socket -> Versio Duo
Changed lines of the file:
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@@
 	(title_block
 		(title "V2 control")
-		(date "2026-03-30")
-		(rev "2026-03-30")
-		(company "Socket")
+		(date "2026-08-27")
+		(rev "2026-08-27")
+		(company "Versio Duo")
+		(comment 1 "Instrument Controller")
 	)
 	(junction
@@
 		(in_pos_files yes)
 		(dnp no)
-		(property "Reference" "#PWR201"
+		(property "Reference" "#PWR041"
 			(at 152.4 71.12 0)
 			(hide yes)
@@
 			(project "control"
 				(path "/6c8448b4-b04d-47e1-934e-e40cbe27a7be/1002ed5a-7984-4d39-a94b-5f1a9a481740"
-					(reference "#PWR201")
+					(reference "#PWR041")
 					(unit 1)
 				)
@@
 		(in_pos_files yes)
 		(dnp no)
-		(property "Reference" "#PWR203"
+		(property "Reference" "#PWR042"
 			(at 152.4 111.76 0)
 			(hide yes)
@@
 			(project "control"
 				(path "/6c8448b4-b04d-47e1-934e-e40cbe27a7be/1002ed5a-7984-4d39-a94b-5f1a9a481740"
-					(reference "#PWR203")
+					(reference "#PWR042")
 					(unit 1)
 				)
@@
 		(dnp no)
 		(fields_autoplaced yes)
-		(property "Reference" "#PWR202"
+		(property "Reference" "#PWR045"
 			(at 172.72 78.74 0)
 			(hide yes)
@@
 			(project "control"
 				(path "/6c8448b4-b04d-47e1-934e-e40cbe27a7be/1002ed5a-7984-4d39-a94b-5f1a9a481740"
-					(reference "#PWR202")
+					(reference "#PWR045")
 					(unit 1)
 				)
@@
 		(in_pos_files yes)
 		(dnp no)
-		(property "Reference" "U201"
+		(property "Reference" "U3"
 			(at 154.3559 72.39 0)
 			(show_name no)
@@
 		(property "Description" ""
 			(at 152.4 90.17 0)
+			(hide yes)
+			(show_name no)
+			(do_not_autoplace no)
+			(effects
+				(font
+					(size 1.27 1.27)
+				)
+			)
+		)
+		(property "Id" "RS485:${SYMBOL_NAME}"
+			(at 152.4 121.92 0)
 			(hide yes)
 			(show_name no)
@@
 			(project "control"
 				(path "/6c8448b4-b04d-47e1-934e-e40cbe27a7be/1002ed5a-7984-4d39-a94b-5f1a9a481740"
-					(reference "U201")
+					(reference "U3")
 					(unit 1)
 				)
@@
 		(in_pos_files yes)
 		(dnp no)
-		(property "Reference" "R201"
+		(property "Reference" "R5"
 			(at 168.91 83.82 0)
 			(show_name no)
@@
 			(hide yes)
 			(show_name yes)
+			(do_not_autoplace no)
+			(effects
+				(font
+					(size 1.27 1.27)
+				)
+			)
+		)
+		(property "Id" "Resistor:${SYMBOL_NAME}"
+			(at 163.83 99.06 0)
+			(hide yes)
+			(show_name no)
 			(do_not_autoplace no)
 			(effects
@@
 			(project "control"
 				(path "/6c8448b4-b04d-47e1-934e-e40cbe27a7be/1002ed5a-7984-4d39-a94b-5f1a9a481740"
-					(reference "R201")
+					(reference "R5")
 					(unit 1)
 				)
@@
 		(in_pos_files yes)
 		(dnp no)
-		(property "Reference" "#PWR204"
+		(property "Reference" "#PWR039"
 			(at 139.7 144.78 0)
 			(hide yes)
@@
 			(project "control"
 				(path "/6c8448b4-b04d-47e1-934e-e40cbe27a7be/1002ed5a-7984-4d39-a94b-5f1a9a481740"
-					(reference "#PWR204")
+					(reference "#PWR039")
 					(unit 1)
 				)
@@
 		(in_pos_files yes)
 		(dnp no)
-		(property "Reference" "J201"
+		(property "Reference" "J5"
 			(at 152.4 133.985 0)
 			(show_name no)
@@
 		(property "Product" "20021112-00010T4LF"
 			(at 152.4 167.64 0)
+			(hide yes)
+			(show_name no)
+			(do_not_autoplace no)
+			(effects
+				(font
+					(size 1.27 1.27)
+				)
+			)
+		)
+		(property "Id" "Header:${SYMBOL_NAME}"
+			(at 152.4 162.56 0)
+			(hide yes)
+			(show_name no)
+			(do_not_autoplace no)
+			(effects
+				(font
+					(size 1.27 1.27)
+				)
+			)
+		)
+		(property "Rating" "1A"
+			(at 152.4 177.8 0)
 			(hide yes)
 			(show_name no)
@@
 			(project "control"
 				(path "/6c8448b4-b04d-47e1-934e-e40cbe27a7be/1002ed5a-7984-4d39-a94b-5f1a9a481740"
-					(reference "J201")
+					(reference "J5")
 					(unit 1)
 				)
@@
 		(in_pos_files yes)
 		(dnp no)
-		(property "Reference" "C201"
+		(property "Reference" "C10"
 			(at 175.26 67.3162 0)
 			(show_name no)
@@
 		(property "Rating" "50V"
 			(at 172.72 92.71 0)
+			(hide yes)
+			(show_name no)
+			(do_not_autoplace no)
+			(effects
+				(font
+					(size 1.27 1.27)
+				)
+			)
+		)
+		(property "Id" "Capacitor:${SYMBOL_NAME}"
+			(at 172.72 85.09 0)
 			(hide yes)
 			(show_name no)
@@
 			(project "control"
 				(path "/6c8448b4-b04d-47e1-934e-e40cbe27a7be/1002ed5a-7984-4d39-a94b-5f1a9a481740"
-					(reference "C201")
+					(reference "C10")
 					(unit 1)
 				)
@@
 		(in_pos_files yes)
 		(dnp no)
-		(property "Reference" "#PWR207"
+		(property "Reference" "#PWR044"
 			(at 165.1 149.86 0)
 			(hide yes)
@@
 			(project "control"
 				(path "/6c8448b4-b04d-47e1-934e-e40cbe27a7be/1002ed5a-7984-4d39-a94b-5f1a9a481740"
-					(reference "#PWR207")
+					(reference "#PWR044")
 					(unit 1)
 				)
@@
 		(in_pos_files yes)
 		(dnp no)
-		(property "Reference" "#PWR206"
+		(property "Reference" "#PWR040"
 			(at 149.86 149.86 0)
 			(hide yes)
@@
 			(project "control"
 				(path "/6c8448b4-b04d-47e1-934e-e40cbe27a7be/1002ed5a-7984-4d39-a94b-5f1a9a481740"
-					(reference "#PWR206")
+					(reference "#PWR040")
 					(unit 1)
 				)
@@
 		(in_pos_files yes)
 		(dnp no)
-		(property "Reference" "#PWR205"
+		(property "Reference" "#PWR043"
 			(at 154.94 144.78 0)
 			(hide yes)
@@
 			(project "control"
 				(path "/6c8448b4-b04d-47e1-934e-e40cbe27a7be/1002ed5a-7984-4d39-a94b-5f1a9a481740"
-					(reference "#PWR205")
+					(reference "#PWR043")
 					(unit 1)
 				)
