File: MIDIIn.kicad_sch (KiCad schematic)
At the start: 6 parts, among them J401 SJ2-25504B-SMT-TR, U401 TLP2361

Commit message: Update TRS socket
Parts:
- J401: value SJ2-25504B-SMT-TR -> SJ2-25404B-SMT-TR; footprint V2_Connector_Audio:CUI_SJ2-25504B-SMT-TR -> V2_Connector_Audio:CUI_SJ2-25404B-SMT-TR; symbol V2_Connector_Audio:SJ2-25504B-SMT-TR -> V2_Connector_Audio:SJ2-25404B-SMT-TR
Connections:
- net Tip: now also J401.2 (T); no longer J401.5 (T)
- net Sleeve: now reaches C401.1, J401.1 (S)
- no-connect marks 3 -> 2
Other:
- moved on the sheet: C401
Changed lines of the file:
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@@
 	(title_block
 		(title "MIDI In")
-		(date "2023-08-08")
+		(date "2024-07-17")
+		(rev "2")
 	)
 	(junction
@@
 	)
 	(no_connect
-		(at 132.08 116.84)
+		(at 129.54 113.03)
 	)
 	(no_connect
-		(at 132.08 109.22)
-	)
-	(no_connect
-		(at 132.08 119.38)
+		(at 129.54 102.87)
 	)
 	(wire
@@
 	(wire
 		(pts
-			(xy 149.86 111.76) (xy 132.08 111.76)
-		)
-		(stroke
-			(width 0)
-			(type default)
-		)
-	)
-	(wire
-		(pts
-			(xy 149.86 107.95) (xy 149.86 111.76)
+			(xy 129.54 107.95) (xy 153.67 107.95)
 		)
 		(stroke
@@
 	(wire
 		(pts
-			(xy 132.08 114.3) (xy 149.86 114.3)
+			(xy 129.54 97.79) (xy 138.43 97.79)
+		)
+		(stroke
+			(width 0)
+			(type default)
+		)
+	)
+	(wire
+		(pts
+			(xy 129.54 118.11) (xy 167.64 118.11)
 		)
 		(stroke
@@
 		)
 	)
-	(wire
-		(pts
-			(xy 149.86 114.3) (xy 149.86 118.11)
-		)
-		(stroke
-			(width 0)
-			(type default)
-		)
-	)
-	(wire
-		(pts
-			(xy 153.67 107.95) (xy 149.86 107.95)
-		)
-		(stroke
-			(width 0)
-			(type default)
-		)
-	)
-	(wire
-		(pts
-			(xy 149.86 118.11) (xy 167.64 118.11)
-		)
-		(stroke
-			(width 0)
-			(type default)
-		)
-	)
 	(polyline
 		(pts
@@
 	)
 	(label "Ring"
-		(at 142.24 111.76 0)
+		(at 132.08 107.95 0)
 		(fields_autoplaced yes)
 		(effects
@@
 	)
 	(label "Tip"
-		(at 142.24 114.3 0)
+		(at 132.08 118.11 0)
+		(fields_autoplaced yes)
+		(effects
+			(font
+				(size 1.27 1.27)
+			)
+			(justify left bottom)
+		)
+	)
+	(label "Sleeve"
+		(at 132.08 97.79 0)
 		(fields_autoplaced yes)
 		(effects
@@
 	(symbol
 		(lib_id "power:GND")
-		(at 137.16 106.68 90)
+		(at 143.51 97.79 90)
 		(unit 1)
 		(exclude_from_sim no)
@@
 		(dnp no)
 		(property "Reference" "#PWR0401"
-			(at 143.51 106.68 0)
+			(at 149.86 97.79 0)
 			(effects
 				(font
@@
 		)
 		(property "Value" "GND"
-			(at 143.51 106.68 90)
+			(at 149.86 97.79 90)
 			(effects
 				(font
@@
 		)
 		(property "Footprint" ""
-			(at 137.16 106.68 0)
+			(at 143.51 97.79 0)
 			(effects
 				(font
@@
 		)
 		(property "Datasheet" ""
-			(at 137.16 106.68 0)
+			(at 143.51 97.79 0)
 			(effects
 				(font
@@
 		)
 		(property "Description" ""
-			(at 137.16 106.68 0)
+			(at 143.51 97.79 0)
 			(effects
 				(font
@@
 	(symbol
 		(lib_id "Device:C_Small")
-		(at 134.62 106.68 90)
+		(at 140.97 97.79 90)
 		(unit 1)
 		(exclude_from_sim no)
@@
 		(dnp no)
 		(property "Reference" "C401"
-			(at 137.1662 99.695 90)
+			(at 143.5162 90.805 90)
 			(effects
 				(font
@@
 		)
 		(property "Value" "0u1"
-			(at 137.1662 102.235 90)
+			(at 143.5162 93.345 90)
 			(effects
 				(font
@@
 		)
 		(property "Footprint" "Capacitor_SMD:C_0603_1608Metric"
-			(at 134.62 106.68 0)
+			(at 140.97 97.79 0)
 			(effects
 				(font
@@
 		)
 		(property "Datasheet" "~"
-			(at 134.62 106.68 0)
+			(at 140.97 97.79 0)
 			(effects
 				(font
@@
 		)
 		(property "Description" ""
-			(at 134.62 106.68 0)
+			(at 140.97 97.79 0)
 			(effects
 				(font
@@
 	)
 	(symbol
-		(lib_id "V2_Connector_Audio:SJ2-25504B-SMT-TR")
-		(at 116.84 113.03 0)
-		(mirror y)
+		(lib_id "V2_Connector_Audio:SJ2-25404B-SMT-TR")
+		(at 116.84 107.95 0)
 		(unit 1)
-		(exclude_from_sim yes)
+		(exclude_from_sim no)
 		(in_bom yes)
 		(on_board yes)
 		(dnp no)
 		(property "Reference" "J401"
-			(at 106.68 98.425 0)
-			(effects
-				(font
-					(size 1.27 1.27)
-				)
-			)
-		)
-		(property "Value" "SJ2-25504B-SMT-TR"
-			(at 114.935 100.965 0)
-			(effects
-				(font
-					(size 1.27 1.27)
-				)
-			)
-		)
-		(property "Footprint" "V2_Connector_Audio:CUI_SJ2-25504B-SMT-TR"
-			(at 140.97 128.27 0)
+			(at 108.966 90.678 0)
+			(effects
+				(font
+					(size 1.27 1.27)
+				)
+			)
+		)
+		(property "Value" "SJ2-25404B-SMT-TR"
+			(at 117.348 92.964 0)
+			(effects
+				(font
+					(size 1.27 1.27)
+				)
+			)
+		)
+		(property "Footprint" "V2_Connector_Audio:CUI_SJ2-25404B-SMT-TR"
+			(at 104.648 128.524 0)
 			(effects
 				(font
@@
 		)
 		(property "Datasheet" ""
-			(at 116.84 113.03 0)
+			(at 116.84 107.95 0)
 			(effects
 				(font
@@
 			)
 		)
-		(property "Description" ""
-			(at 116.84 113.03 0)
-			(effects
-				(font
-					(size 1.27 1.27)
-				)
-				(hide yes)
-			)
-		)
-		(property "Sim.Enable" "0"
-			(at 116.84 113.03 0)
-			(effects
-				(font
-					(size 1.27 1.27)
-				)
+		(property "Description" "SJ2-35464B-SMT-TR"
+			(at 108.712 131.064 0)
+			(effects
+				(font
+					(size 1.27 1.27)
+				)
+				(justify left bottom)
 				(hide yes)
 			)
@@
 		(pin "4"
 		)
-		(pin "5"
-		)
 		(instances

Commit message: Refresh
Parts:
- U401: footprint Package_SO:SO-5_4.4x3.6mm_P1.27mm -> Package_SO:SO-5-6_4.55x3.7mm_P1.27mm
- renumbered C402 to C401, C401 to C402
Changed lines of the file:
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@@
 (kicad_sch
-	(version 20231120)
+	(version 20250114)
 	(generator "eeschema")
-	(generator_version "8.0")
+	(generator_version "9.0")
 	(paper "A4")
 	(title_block
 		(title "MIDI In")
-		(date "2024-07-17")
-		(rev "2")
+		(date "2025-10-27")
+		(rev "3")
 	)
 	(junction
@@
 	(label "Ring"
 		(at 132.08 107.95 0)
-		(fields_autoplaced yes)
 		(effects
 			(font
@@
 	(label "Tip"
 		(at 132.08 118.11 0)
-		(fields_autoplaced yes)
 		(effects
 			(font
@@
 	(label "Sleeve"
 		(at 132.08 97.79 0)
-		(fields_autoplaced yes)
 		(effects
 			(font
@@
 		(shape output)
 		(at 207.01 113.03 0)
-		(fields_autoplaced yes)
 		(effects
 			(font
@@
 		(on_board yes)
 		(dnp no)
-		(property "Reference" "#PWR0403"
+		(property "Reference" "#PWR0404"
 			(at 187.96 129.54 0)
 			(effects
@@
 			(project "control"
 				(path "/6c8448b4-b04d-47e1-934e-e40cbe27a7be/ae0f3fb3-3b08-46e7-ba0a-341c37aaf317"
-					(reference "#PWR0403")
+					(reference "#PWR0404")
 					(unit 1)
 				)
@@
 		(on_board yes)
 		(dnp no)
-		(property "Reference" "#PWR0401"
+		(property "Reference" "#PWR0402"
 			(at 149.86 97.79 0)
 			(effects
@@
 			(project "control"
 				(path "/6c8448b4-b04d-47e1-934e-e40cbe27a7be/ae0f3fb3-3b08-46e7-ba0a-341c37aaf317"
-					(reference "#PWR0401")
+					(reference "#PWR0402")
 					(unit 1)
 				)
@@
 		(on_board yes)
 		(dnp no)
-		(property "Reference" "C401"
+		(property "Reference" "C402"
 			(at 143.5162 90.805 90)
 			(effects
@@
 			(project "control"
 				(path "/6c8448b4-b04d-47e1-934e-e40cbe27a7be/ae0f3fb3-3b08-46e7-ba0a-341c37aaf317"
-					(reference "C401")
+					(reference "C402")
 					(unit 1)
 				)
@@
 			)
 		)
-		(property "Footprint" "Package_SO:SO-5_4.4x3.6mm_P1.27mm"
+		(property "Footprint" "Package_SO:SO-5-6_4.55x3.7mm_P1.27mm"
 			(at 170.18 125.73 0)
 			(effects
@@
 		(on_board yes)
 		(dnp no)
-		(property "Reference" "C402"
+		(property "Reference" "C401"
 			(at 196.85 93.3512 0)
 			(effects
@@
 			(project "control"
 				(path "/6c8448b4-b04d-47e1-934e-e40cbe27a7be/ae0f3fb3-3b08-46e7-ba0a-341c37aaf317"
-					(reference "C402")
+					(reference "C401")
 					(unit 1)
 				)
@@
 		(on_board yes)
 		(dnp no)
-		(property "Reference" "#PWR0402"
+		(property "Reference" "#PWR0401"
 			(at 187.96 96.52 0)
 			(effects
@@
 			(project "control"
 				(path "/6c8448b4-b04d-47e1-934e-e40cbe27a7be/ae0f3fb3-3b08-46e7-ba0a-341c37aaf317"
-					(reference "#PWR0402")
+					(reference "#PWR0401")
 					(unit 1)
 				)
@@
 		(on_board yes)
 		(dnp no)
-		(property "Reference" "#PWR0404"
+		(property "Reference" "#PWR0403"
 			(at 193.04 104.14 0)
 			(effects
@@
 			(project "control"
 				(path "/6c8448b4-b04d-47e1-934e-e40cbe27a7be/ae0f3fb3-3b08-46e7-ba0a-341c37aaf317"
-					(reference "#PWR0404")
-					(unit 1)
-				)
+					(reference "#PWR0403")
+					(unit 1)
+				)
