File: MIDIIn.kicad_sch (KiCad schematic)
At the start: 6 parts, among them J401 SJ2-25404B-SMT-TR, U401 TLP2361

Commit message: Update
Parts:
- C11: renamed from C402; Id (none) -> Capacitor:${SYMBOL_NAME}
- C12: renamed from C401; Id (none) -> Capacitor:${SYMBOL_NAME}
- D4: renamed from D401; Id (none) -> Diode:${SYMBOL_NAME}
- J9: renamed from J401; Id (none) -> Audio:${SYMBOL_NAME}; Rating (none) -> 2.5mm
- R6: renamed from R401; Id (none) -> Resistor:${SYMBOL_NAME}
- U5: renamed from U401; Id (none) -> Optocoupler:${SYMBOL_NAME}; Rating (none) -> 15Mbps
Other:
- company: (none) -> Versio Duo
Changed lines of the file:
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@@
 	(title_block
 		(title "V2 control")
-		(date "2026-03-30")
-		(rev "2026-03-30")
+		(date "2026-08-27")
+		(rev "2026-08-27")
+		(company "Versio Duo")
+		(comment 1 "Instrument Controller")
 	)
