File: PowerSupply.kicad_sch (KiCad schematic)
At the start: 6 parts, among them U501 TPSM33620S5QRDNRQ1

Commit message: Update
Parts:
- C13: renamed from C501; Id (none) -> Capacitor:${SYMBOL_NAME}
- C14: renamed from C502; Id (none) -> Capacitor:${SYMBOL_NAME}
- C15: renamed from C505; Id (none) -> Capacitor:${SYMBOL_NAME}
- C16: renamed from C503; Id (none) -> Capacitor:${SYMBOL_NAME}
- C17: renamed from C504; Id (none) -> Capacitor:${SYMBOL_NAME}
- U6: renamed from U501; Id (none) -> DCDC:${SYMBOL_NAME}
Other:
- company: +5V -> Versio Duo
Changed lines of the file:
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@@
 	(title_block
 		(title "V2 control")
-		(date "2026-03-30")
-		(rev "2026-03-30")
-		(company "+5V")
+		(date "2026-08-27")
+		(rev "2026-08-27")
+		(company "Versio Duo")
+		(comment 1 "Instrument Controller")
 	)
 	(junction
@@
 		(in_pos_files yes)
 		(dnp no)
-		(property "Reference" "#PWR504"
+		(property "Reference" "#PWR059"
 			(at 194.31 107.95 0)
 			(hide yes)
@@
 			(project "control"
 				(path "/6c8448b4-b04d-47e1-934e-e40cbe27a7be/24a9dc0c-cb3c-464a-a734-f09bf949d71a"
-					(reference "#PWR504")
+					(reference "#PWR059")
 					(unit 1)
 				)
@@
 		(in_pos_files yes)
 		(dnp no)
-		(property "Reference" "#PWR507"
+		(property "Reference" "#PWR056"
 			(at 127 106.68 0)
 			(hide yes)
@@
 			(project "control"
 				(path "/6c8448b4-b04d-47e1-934e-e40cbe27a7be/24a9dc0c-cb3c-464a-a734-f09bf949d71a"
-					(reference "#PWR507")
+					(reference "#PWR056")
 					(unit 1)
 				)
@@
 		(in_pos_files yes)
 		(dnp no)
-		(property "Reference" "U501"
+		(property "Reference" "U6"
 			(at 151.13 88.9 0)
 			(show_name no)
@@
 		(property "Rating" "2A"
 			(at 158.75 154.94 0)
+			(hide yes)
+			(show_name no)
+			(do_not_autoplace no)
+			(effects
+				(font
+					(size 1.27 1.27)
+				)
+			)
+		)
+		(property "Id" "DCDC:${SYMBOL_NAME}"
+			(at 158.75 148.59 0)
 			(hide yes)
 			(show_name no)
@@
 			(project "control"
 				(path "/6c8448b4-b04d-47e1-934e-e40cbe27a7be/24a9dc0c-cb3c-464a-a734-f09bf949d71a"
-					(reference "U501")
+					(reference "U6")
 					(unit 1)
 				)
@@
 		(in_pos_files yes)
 		(dnp no)
-		(property "Reference" "#PWR503"
+		(property "Reference" "#PWR055"
 			(at 119.38 107.95 0)
 			(hide yes)
@@
 			(project "control"
 				(path "/6c8448b4-b04d-47e1-934e-e40cbe27a7be/24a9dc0c-cb3c-464a-a734-f09bf949d71a"
-					(reference "#PWR503")
+					(reference "#PWR055")
 					(unit 1)
 				)
@@
 		(in_pos_files yes)
 		(dnp no)
-		(property "Reference" "C501"
+		(property "Reference" "C13"
 			(at 110.49 97.79 0)
 			(show_name no)
@@
 		)
 		(property "Manufacturer" "TDK"
+			(at 107.95 114.3 0)
+			(hide yes)
+			(show_name no)
+			(do_not_autoplace no)
+			(effects
+				(font
+					(size 1.27 1.27)
+				)
+			)
+		)
+		(property "Id" "Capacitor:${SYMBOL_NAME}"
 			(at 107.95 114.3 0)
 			(hide yes)
@@
 			(project "control"
 				(path "/6c8448b4-b04d-47e1-934e-e40cbe27a7be/24a9dc0c-cb3c-464a-a734-f09bf949d71a"
-					(reference "C501")
+					(reference "C13")
 					(unit 1)
 				)
@@
 		(in_pos_files yes)
 		(dnp no)
-		(property "Reference" "C505"
+		(property "Reference" "C15"
 			(at 134.366 110.998 90)
 			(show_name no)
@@
 		(property "Rating" "50V"
 			(at 113.03 106.68 0)
+			(hide yes)
+			(show_name no)
+			(do_not_autoplace no)
+			(effects
+				(font
+					(size 1.27 1.27)
+				)
+			)
+		)
+		(property "Id" "Capacitor:${SYMBOL_NAME}"
+			(at 120.65 106.68 0)
 			(hide yes)
 			(show_name no)
@@
 			(project "control"
 				(path "/6c8448b4-b04d-47e1-934e-e40cbe27a7be/24a9dc0c-cb3c-464a-a734-f09bf949d71a"
-					(reference "C505")
+					(reference "C15")
 					(unit 1)
 				)
@@
 		(in_pos_files yes)
 		(dnp no)
-		(property "Reference" "C503"
+		(property "Reference" "C16"
 			(at 196.85 97.79 0)
 			(show_name no)
@@
 		)
 		(property "Manufacturer" "TDK"
+			(at 194.31 114.3 0)
+			(hide yes)
+			(show_name no)
+			(do_not_autoplace no)
+			(effects
+				(font
+					(size 1.27 1.27)
+				)
+			)
+		)
+		(property "Id" "Capacitor:${SYMBOL_NAME}"
 			(at 194.31 114.3 0)
 			(hide yes)
@@
 			(project "control"
 				(path "/6c8448b4-b04d-47e1-934e-e40cbe27a7be/24a9dc0c-cb3c-464a-a734-f09bf949d71a"
-					(reference "C503")
+					(reference "C16")
 					(unit 1)
 				)
@@
 		(in_pos_files yes)
 		(dnp no)
-		(property "Reference" "C502"
+		(property "Reference" "C14"
 			(at 121.92 97.79 0)
 			(show_name no)
@@
 		(property "Rating" "50V"
 			(at 119.38 121.92 0)
+			(hide yes)
+			(show_name no)
+			(do_not_autoplace no)
+			(effects
+				(font
+					(size 1.27 1.27)
+				)
+			)
+		)
+		(property "Id" "Capacitor:${SYMBOL_NAME}"
+			(at 119.38 114.3 0)
 			(hide yes)
 			(show_name no)
@@
 			(project "control"
 				(path "/6c8448b4-b04d-47e1-934e-e40cbe27a7be/24a9dc0c-cb3c-464a-a734-f09bf949d71a"
-					(reference "C502")
+					(reference "C14")
 					(unit 1)
 				)
@@
 		(in_pos_files yes)
 		(dnp no)
-		(property "Reference" "#PWR502"
+		(property "Reference" "#PWR054"
 			(at 107.95 107.95 0)
 			(hide yes)
@@
 			(project "control"
 				(path "/6c8448b4-b04d-47e1-934e-e40cbe27a7be/24a9dc0c-cb3c-464a-a734-f09bf949d71a"
-					(reference "#PWR502")
+					(reference "#PWR054")
 					(unit 1)
 				)
@@
 		(in_pos_files yes)
 		(dnp no)
-		(property "Reference" "#PWR509"
+		(property "Reference" "#PWR057"
 			(at 139.7 111.76 0)
 			(hide yes)
@@
 			(project "control"
 				(path "/6c8448b4-b04d-47e1-934e-e40cbe27a7be/24a9dc0c-cb3c-464a-a734-f09bf949d71a"
-					(reference "#PWR509")
+					(reference "#PWR057")
 					(unit 1)
 				)
@@
 		(in_pos_files yes)
 		(dnp no)
-		(property "Reference" "#PWR505"
+		(property "Reference" "#PWR061"
 			(at 205.74 107.95 0)
 			(hide yes)
@@
 			(project "control"
 				(path "/6c8448b4-b04d-47e1-934e-e40cbe27a7be/24a9dc0c-cb3c-464a-a734-f09bf949d71a"
-					(reference "#PWR505")
+					(reference "#PWR061")
 					(unit 1)
 				)
@@
 		(in_pos_files yes)
 		(dnp no)
-		(property "Reference" "#PWR501"
+		(property "Reference" "#PWR060"
 			(at 205.74 100.33 0)
 			(hide yes)
@@
 			(project "control"
 				(path "/6c8448b4-b04d-47e1-934e-e40cbe27a7be/24a9dc0c-cb3c-464a-a734-f09bf949d71a"
-					(reference "#PWR501")
+					(reference "#PWR060")
 					(unit 1)
 				)
@@
 		(in_pos_files yes)
 		(dnp no)
-		(property "Reference" "#PWR508"
+		(property "Reference" "#PWR058"
 			(at 158.75 123.19 0)
 			(hide yes)
@@
 			(project "control"
 				(path "/6c8448b4-b04d-47e1-934e-e40cbe27a7be/24a9dc0c-cb3c-464a-a734-f09bf949d71a"
-					(reference "#PWR508")
+					(reference "#PWR058")
 					(unit 1)
 				)
@@
 		(in_pos_files yes)
 		(dnp no)
-		(property "Reference" "C504"
+		(property "Reference" "C17"
 			(at 208.28 97.79 0)
 			(show_name no)
@@
 		)
 		(property "Manufacturer" "TDK"
+			(at 205.74 114.3 0)
+			(hide yes)
+			(show_name no)
+			(do_not_autoplace no)
+			(effects
+				(font
+					(size 1.27 1.27)
+				)
+			)
+		)
+		(property "Id" "Capacitor:${SYMBOL_NAME}"
 			(at 205.74 114.3 0)
 			(hide yes)
@@
 			(project "control"
 				(path "/6c8448b4-b04d-47e1-934e-e40cbe27a7be/24a9dc0c-cb3c-464a-a734-f09bf949d71a"
-					(reference "C504")
+					(reference "C17")
 					(unit 1)
 				)
