File: control.kicad_pcb (KiCad board)
At the start: 4 copper layers, 60 x 35 mm, 67 parts, among them J101 Cortex, J102 DX07S016JA3, J103 WAGO 2065-100, J104 WAGO 2065-100, J201 2x05_Horizontal, J301 WAGO 2065-100, J302 WAGO 2065-100, J303 WAGO 2065-100, J401 SJ2-25404B-SMT-TR, SW101 SKSG, SW102 SKSG, U101 TPS78433QWDRBRQ1, U102 ATSAMD51G, U301 74AHC1G125, U401 TLP2361, U501 TPSM33620S5QRDNRQ1, Y101 32k768

Commit message: Update
Parts:
- added C801: 0u1, V2_Capacitor_SMD:C_1608, F.Cu at (147.0, 93.0)
- C1: renamed from C108; footprint V2_Capacitor_SMD:C_0603 -> V2_Capacitor_SMD:C_1608
- C10: renamed from C201; footprint V2_Capacitor_SMD:C_0603 -> V2_Capacitor_SMD:C_1608
- C11: renamed from C402; footprint V2_Capacitor_SMD:C_0603 -> V2_Capacitor_SMD:C_1608
- C12: renamed from C401; footprint V2_Capacitor_SMD:C_0603 -> V2_Capacitor_SMD:C_1608
- C13: renamed from C501; footprint V2_Capacitor_SMD:C_1210 -> V2_Capacitor_SMD:C_3225
- C14: renamed from C502; footprint V2_Capacitor_SMD:C_0603 -> V2_Capacitor_SMD:C_1608
- C15: renamed from C505; footprint V2_Capacitor_SMD:C_0603 -> V2_Capacitor_SMD:C_1608
- C16: renamed from C503; footprint V2_Capacitor_SMD:C_1210 -> V2_Capacitor_SMD:C_3225
- C17: renamed from C504; footprint V2_Capacitor_SMD:C_1210 -> V2_Capacitor_SMD:C_3225
- C2: renamed from C109; footprint V2_Capacitor_SMD:C_0603 -> V2_Capacitor_SMD:C_1608
- C3: renamed from C101; footprint V2_Capacitor_SMD:C_0603 -> V2_Capacitor_SMD:C_1608
- C4: renamed from C102; footprint V2_Capacitor_SMD:C_0603 -> V2_Capacitor_SMD:C_1608
- C5: renamed from C103; footprint V2_Capacitor_SMD:C_0603 -> V2_Capacitor_SMD:C_1608
- C6: renamed from C104; footprint V2_Capacitor_SMD:C_0603 -> V2_Capacitor_SMD:C_1608
- C7: renamed from C105; footprint V2_Capacitor_SMD:C_0603 -> V2_Capacitor_SMD:C_1608
- C8: renamed from C106; footprint V2_Capacitor_SMD:C_0805 -> V2_Capacitor_SMD:C_2012
- C9: renamed from C107; footprint V2_Capacitor_SMD:C_0805 -> V2_Capacitor_SMD:C_2012
- D1: renamed from D103; footprint V2_LED:LED_0603 -> V2_LED:LED_1608
- H1: renamed from SPACER101; value 9774030243 -> 2mm; footprint V2_Spacer_Wurth:9774030243 -> V2_Mechanical:MountingHole_2mm
- H2: renamed from SPACER102; value 9774030243 -> 2mm; footprint V2_Spacer_Wurth:9774030243 -> V2_Mechanical:MountingHole_2mm
- H3: renamed from SPACER103; value 9774030243 -> 2mm; footprint V2_Spacer_Wurth:9774030243 -> V2_Mechanical:MountingHole_2mm
- H4: renamed from SPACER104; value 9774030243 -> 2mm; footprint V2_Spacer_Wurth:9774030243 -> V2_Mechanical:MountingHole_2mm
- INFO2: renamed from INFO101; value Layer_Numbers -> Layer_Numbers-4; footprint V2_Production:Layer_Numbers -> V2_Production:Layer_Numbers-4
- R1: renamed from R105; footprint V2_Resistor_SMD:R_0603 -> V2_Resistor_SMD:R_1608
- R2: renamed from R101; footprint V2_Resistor_SMD:R_0603 -> V2_Resistor_SMD:R_1608
- R3: renamed from R103; footprint V2_Resistor_SMD:R_0603 -> V2_Resistor_SMD:R_1608
- R4: renamed from R104; footprint V2_Resistor_SMD:R_0603 -> V2_Resistor_SMD:R_1608
- R5: renamed from R201; footprint V2_Resistor_SMD:R_0603 -> V2_Resistor_SMD:R_1608
- R6: renamed from R401; footprint V2_Resistor_SMD:R_0603 -> V2_Resistor_SMD:R_1608
- TVS2: renamed from TVS101; footprint V2_Diode_SMD:D_0603 -> V2_Diode_SMD:D_1608
- moved ICON2 1.03 mm to (170.5, 87.0)
- moved U4 1.00 mm to (147.0, 90.5)
- moved ESD1 0.75 mm to (130.8, 104.2)
- moved C8 0.71 mm to (135.8, 110.8)
- moved C9 0.71 mm to (135.8, 104.2)
- moved TVS2 0.71 mm to (135.8, 112.5)
- moved U2 0.71 mm to (135.8, 107.5)
- moved ICON4 0.25 mm to (136.5, 89.8)
- moved ICON5 0.25 mm to (150.8, 89.5)
- moved ICON6 0.25 mm to (143.5, 89.8)
- renumbered D101 to D2, D102 to D3, D401 to D4, ESD101 to ESD1, FID101 to FID1, FID102 to FID2, FID103 to FID3, H101 to H5, H102 to H6, ICON103 to ICON1, ICON105 to ICON2, ICON101 to ICON3, ICON102 to ICON4, ICON104 to ICON5, ICON106 to ICON6, INFO102 to INFO1, J103 to J1, J104 to J2, J101 to J3, J102 to J4, J201 to J5, J301 to J6, J302 to J7, J303 to J8, J401 to J9, PLUG101 to PLUG1, SW102 to SW1, SW101 to SW2, SWB101 to SWB1, TVS102 to TVS1, U102 to U1, U101 to U2, U201 to U3, U301 to U4, U401 to U5, U501 to U6, Y101 to Y1
Connections:
- ESD1 pad 2: unconnected-(ESD101-D2-Pad2) -> /USB-
- ESD1 pad 3: unconnected-(ESD101-D1-Pad3) -> /USB+
- J4 pad V: /+VBUS -> unconnected-(J4-VBUS-PadV)
- U2 pad 6: unconnected-(U101-Pad6) -> +5V
Routing:
- net +5V: track 15.2 -> 134.8 mm, vias 18 -> 17
- net +3V3: track 27.8 -> 97.2 mm
- net /+VBUS: track 7.15 -> 0.00 mm, vias 2 -> 0
- net /LED-Data: track 17.0 -> 19.2 mm
- net /Link Socket/TX-Y: track 15.3 -> 13.3 mm
- net /Button-LED: track 8.33 -> 10.1 mm
- net /USB-: track 36.9 -> 38.5 mm, vias 3 -> 2
- net /USB+: track 34.0 -> 35.1 mm, vias 3 -> 2
- net GND: track 31.6 -> 32.7 mm, vias 68 -> 69
- net /LED Strip/WS2812-data: track 6.43 -> 5.36 mm
- net /Link Socket/TX-Z: track 15.6 -> 14.8 mm
- net Net-(D4-K): track 5.82 -> 5.28 mm
- removed copper zone on In2.Cu, net +3V3
- removed copper zone on In2.Cu, net +5V
- removed copper zone on B.Cu, net GND
