File: control.kicad_sch (KiCad schematic)
At the start: 47 parts, among them J101 Cortex, J102 DX07S016JA3, J103 WAGO 2065-100, J104 WAGO 2065-100, SW101 SKSG, SW102 SKSG, U101 TPS78433QWDRBRQ1, U102 ATSAMD51G, Y101 32k768

Commit message: Update
Parts:
- C1: renamed from C108; Id (none) -> Capacitor:${SYMBOL_NAME}
- C2: renamed from C109; Id (none) -> Capacitor:${SYMBOL_NAME}
- C3: renamed from C101; Id (none) -> Capacitor:${SYMBOL_NAME}
- C4: renamed from C102; Id (none) -> Capacitor:${SYMBOL_NAME}
- C5: renamed from C103; Id (none) -> Capacitor:${SYMBOL_NAME}
- C6: renamed from C104; Id (none) -> Capacitor:${SYMBOL_NAME}
- C7: renamed from C105; Id (none) -> Capacitor:${SYMBOL_NAME}
- C8: renamed from C106; Id (none) -> Capacitor:${SYMBOL_NAME}
- C9: renamed from C107; Id (none) -> Capacitor:${SYMBOL_NAME}
- D1: renamed from D103; footprint V2_LED:LED_0603 -> V2_LED:LED_1608; Id (none) -> LED:${SYMBOL_NAME}; Rating (none) -> 605nm
- D2: renamed from D101; Id (none) -> LED:${SYMBOL_NAME}; Rating (none) -> 15mA
- D3: renamed from D102; Id (none) -> LED:${SYMBOL_NAME}; Rating (none) -> 15mA
- ESD1: renamed from ESD101; Id (none) -> ESD:${SYMBOL_NAME}; Rating (none) -> 20kV
- H1: renamed from SPACER101; value 9774030243 -> 2mm; footprint V2_Spacer_Wurth:9774030243 -> V2_Mechanical:MountingHole_2mm; symbol V2_Spacer_Wurth:9774030243 -> V2_Mechanical:MountingHole_2mm; now left out of the parts list
- H2: renamed from SPACER102; value 9774030243 -> 2mm; footprint V2_Spacer_Wurth:9774030243 -> V2_Mechanical:MountingHole_2mm; symbol V2_Spacer_Wurth:9774030243 -> V2_Mechanical:MountingHole_2mm; now left out of the parts list
- H3: renamed from SPACER103; value 9774030243 -> 2mm; footprint V2_Spacer_Wurth:9774030243 -> V2_Mechanical:MountingHole_2mm; symbol V2_Spacer_Wurth:9774030243 -> V2_Mechanical:MountingHole_2mm; now left out of the parts list
- H4: renamed from SPACER104; value 9774030243 -> 2mm; footprint V2_Spacer_Wurth:9774030243 -> V2_Mechanical:MountingHole_2mm; symbol V2_Spacer_Wurth:9774030243 -> V2_Mechanical:MountingHole_2mm; now left out of the parts list
- INFO2: renamed from INFO101; value Layer_Numbers -> Layer_Numbers-4; footprint V2_Production:Layer_Numbers -> V2_Production:Layer_Numbers-4; symbol V2_Production:Layer_Numbers -> V2_Production:Layer_Numbers-4
- J1: renamed from J103; Id (none) -> WAGO:${SYMBOL_NAME}; Rating (none) -> 9A
- J2: renamed from J104; Id (none) -> WAGO:${SYMBOL_NAME}; Rating (none) -> 9A
- J4: renamed from J102; Id (none) -> USB:${SYMBOL_NAME}; Rating (none) -> USB2.0
- R1: renamed from R105; Id (none) -> Resistor:${SYMBOL_NAME}
- R2: renamed from R101; Id (none) -> Resistor:${SYMBOL_NAME}
- R3: renamed from R103; Id (none) -> Resistor:${SYMBOL_NAME}
- R4: renamed from R104; Id (none) -> Resistor:${SYMBOL_NAME}
- SW1: renamed from SW102; Id (none) -> Button:${SYMBOL_NAME}
- SW2: renamed from SW101; Id (none) -> Button:${SYMBOL_NAME}
- TVS1: renamed from TVS102; Id (none) -> Diode:${SYMBOL_NAME}
- TVS2: renamed from TVS101; footprint V2_Diode_SMD:D_0603 -> V2_Diode_SMD:D_1608; Id (none) -> Diode:${SYMBOL_NAME}
- U1: renamed from U102; Id (none) -> MCU:${SYMBOL_NAME}; Rating (none) -> Cortex-M4F
- U2: renamed from U101; Id (none) -> LDO:${SYMBOL_NAME}; Rating (none) -> 300mA
- Y1: renamed from Y101; Id (none) -> Crystal:${SYMBOL_NAME}; Rating (none) -> 10ppm
- renumbered FID101 to FID1, FID102 to FID2, FID103 to FID3, H101 to H5, H102 to H6, ICON103 to ICON1, ICON105 to ICON2, ICON101 to ICON3, ICON102 to ICON4, ICON104 to ICON5, ICON106 to ICON6, INFO102 to INFO1, J101 to J3, PLUG101 to PLUG1, SWB101 to SWB1
Connections:
- net +5V: now also U2.6 (EN)
- net GND: no longer H1.1, H2.1, H3.1, H4.1
- net USB+: now also ESD1.3 (D1)
- net USB-: now also ESD1.2 (D2)
- net +VBUS: no longer names the net of J4.V (VBUS)
- no-connect marks 27 -> 26
Other:
- moved on the sheet: ICON1, ICON2, ICON3, ICON4, ICON5, ICON6, INFO1, INFO2, PLUG1, SWB1
